File: YC265A0-Debug/AUDIO_IO.kicad_sch (KiCad schematic)
At the start: 7 parts, among them U1 TLV320AIC3204

Commit message: sample 1
Parts:
- added C10, C9: 0.1uF, Capacitor_SMD:C_0603_1608Metric_Pad1.08x0.95mm_HandSolder, symbol Device:C
- added C11, C12: 10u, Capacitor_SMD:C_0603_1608Metric_Pad1.08x0.95mm_HandSolder, symbol Device:C
- added C7, C8: 2.2nF, Capacitor_SMD:C_0603_1608Metric_Pad1.08x0.95mm_HandSolder, symbol Device:C
- added J2: AUDIO-OUT, Connector_Audio:Jack_3.5mm_PJ320D_Horizontal, symbol Connector_Audio:AudioJack4
- added J3: MIC-1, Connector_Audio:Jack_3.5mm_PJ320D_Horizontal, symbol Connector_Audio:AudioJack4
- added J4: MIC-2, Connector_Audio:Jack_3.5mm_PJ320D_Horizontal, symbol Connector_Audio:AudioJack4
- added JP1: MICBIAS, Connector_PinHeader_2.54mm:PinHeader_1x02_P2.54mm_Vertical, symbol Jumper:Jumper_2_Open
- added JP2: AVDD_SPLIT, Connector_PinHeader_2.54mm:PinHeader_1x02_P2.54mm_Vertical, symbol Jumper:Jumper_2_Open
- added R1, R2: 470, Resistor_SMD:R_0603_1608Metric_Pad0.98x0.95mm_HandSolder, symbol Device:R
- added R3, R4: 2.7k, Resistor_SMD:R_0603_1608Metric_Pad0.98x0.95mm_HandSolder, symbol Device:R
- added U3: LM1117MP-3.3, Package_TO_SOT_SMD:SOT-223-3_TabPin2, symbol Regulator_Linear:LM1117MP-3.3
- C1, C2, C3, C4, C5, C6: footprint (none) -> Capacitor_SMD:C_0603_1608Metric_Pad1.08x0.95mm_HandSolder
- U1: footprint (none) -> Package_DFN_QFN:VQFN-32-1EP_5x5mm_P0.5mm_EP3.5x3.5mm
Connections:
- net +3.3V: now also JP2.1 (A); no longer U1.30 (LDO_SELECT)
- net GND: now also C11.1, C12.1, C7.2, C8.1, J2.S, J3.S, J4.S, U3.1 (GND)
- net MIC1_IN: now reaches U1.13 (IN1_L)
- net MIC1_IN: now also C10.2
- net MIC2_IN: now reaches U1.14 (IN1_R)
- net MIC2_IN: now also C9.2
- net at U1.19 (MICBIAS): now also JP1.1 (A)
- net LINEOUT_L: now reaches U1.22 (LOL)
- net LINEOUT_L: now also R1.1
- net LINEOUT_R: now reaches U1.23 (LOR)
- net LINEOUT_R: now also R2.2
- net CODEC-BCLK renamed BCLK
- net CODEC-DIN renamed DIN
- net CODEC-DOUT renamed DOUT
- net CODEC-MCLK renamed MCLK
- net CODEC-RESET renamed RESET
- net CODEC-SCL renamed SCL
- net CODEC-SDA renamed SDA
- net CODEC-WCLK renamed WCLK
- new net: C7.1, J2.T, R1.2
- new net: C10.1, J3.T, R4.1
- new net: C9.1, J4.T, R3.1
- new net: C8.2, J2.R1, R2.1
- new net +3.3VA: C11.2, JP2.2 (B), U1.30 (LDO_SELECT), U3.2 (VO)
- new net +5V: C12.2, U3.3 (VI)
- new net MICBIAS: JP1.2 (B), R3.2, R4.2
- no-connect marks 9 -> 14
Other:
- title: (none) -> DAC/ADC IO parts
- moved on the sheet: C1, C2, C3
