File: YC265A0-Debug/MCU.kicad_sch (KiCad schematic)
At the start: 0 parts

Commit message: sample 1
Parts:
- added C13: 0.01u, Capacitor_SMD:C_0603_1608Metric_Pad1.08x0.95mm_HandSolder, symbol Device:C
- added D1: LED1, LED_SMD:LED_0603_1608Metric_Pad1.05x0.95mm_HandSolder, symbol Device:LED
- added D2: LED2, LED_SMD:LED_0603_1608Metric_Pad1.05x0.95mm_HandSolder, symbol Device:LED
- added D3: LED3, LED_SMD:LED_0603_1608Metric_Pad1.05x0.95mm_HandSolder, symbol Device:LED
- added D4: LED4, LED_SMD:LED_0603_1608Metric_Pad1.05x0.95mm_HandSolder, symbol Device:LED
- added J5: USB, Connector_USB:USB_C_Receptacle_Palconn_UTC16-G, symbol Connector:USB_C_Receptacle_USB2.0_14P
- added J7: Conn_01x02_Pin, Connector_PinHeader_2.54mm:PinHeader_1x02_P2.54mm_Horizontal, symbol Connector:Conn_01x02_Pin
- added R10, R11, R8, R9: 1k, Resistor_SMD:R_0603_1608Metric_Pad0.98x0.95mm_HandSolder, symbol Device:R
- added R12, R13: 3.3k, Resistor_SMD:R_0603_1608Metric_Pad0.98x0.95mm_HandSolder, symbol Device:R
- added R5, R6: 5.1k, Resistor_SMD:R_0603_1608Metric_Pad0.98x0.95mm_HandSolder, symbol Device:R
- added R7: 10k, Resistor_SMD:R_0603_1608Metric_Pad0.98x0.95mm_HandSolder, symbol Device:R
- added SW1: RESET, Button_Switch_THT:SW_PUSH_6mm_H8mm, symbol Switch:SW_Push
- added SW2: FLASH, Button_Switch_THT:SW_PUSH_6mm_H8mm, symbol Switch:SW_Push
- added U2: ESP32-S3-WROOM-1, RF_Module:ESP32-S3-WROOM-1, symbol RF_Module:ESP32-S3-WROOM-1
Connections:
- new net: D1.2 (A), R8.2
- new net: D4.2 (A), R11.2
- new net: D3.2 (A), R10.2
- new net: D2.2 (A), R9.2
- new net: J5.B5 (CC2), R6.1
- new net: J5.A5 (CC1), R5.1
- new net +3.3V: R12.2, R13.2, R7.1, U2.2 (3V3)
- new net +5V: J5.A4 (VBUS), J5.A9 (VBUS), J5.B4 (VBUS), J5.B9 (VBUS)
- new net CODEC_RESET: U2.31 (IO38)
- new net DEBUG_RX: J7.2 (Pin_2), U2.36 (RXD0)
- new net DEBUG_TX: J7.1 (Pin_1), U2.37 (TXD0)
- new net EN: C13.1, R7.2, SW1.1, U2.3 (EN)
- new net FLASH: SW2.1, U2.27 (IO0)
- new net GND: C13.2, D1.1 (K), D2.1 (K), D3.1 (K), D4.1 (K), J5.A1 (GND), J5.A12 (GND), J5.B1 (GND), J5.B12 (GND), J5.S1 (SHIELD), R5.2, R6.2, SW1.2, SW2.2, U2.1 (GND), U2.40 (GND), U2.41 (GND)
- new net I2C_SCL: R13.1, U2.26 (IO45)
- new net I2C_SDA: R12.1, U2.25 (IO48)
- new net I2S_BCLK: U2.22 (IO14)
- new net I2S_IN: U2.4 (IO4)
- new net I2S_MCLK: U2.21 (IO13)
- new net I2S_OUT1: U2.20 (IO12)
- new net I2S_OUT2: U2.19 (IO11)
- new net I2S_OUT3: U2.18 (IO10)
- new net I2S_WCLK: U2.23 (IO21)
- new net KDSP_RX: U2.17 (IO9)
- new net KDSP_TX: U2.16 (IO46)
- new net LED1: R8.1, U2.32 (IO39)
- new net LED2: R9.1, U2.33 (IO40)
- new net LED3: R10.1, U2.34 (IO41)
- new net LED4: R11.1, U2.35 (IO42)
- new net SDSP_RX: U2.11 (IO18)
- new net SDSP_TX: U2.10 (IO17)
- new net TG1A_TX: U2.15 (IO3)
- new net TG1B_TX: U2.7 (IO7)
- new net TG1_RX: U2.8 (IO15)
- new net TG2A_TX: U2.9 (IO16)
- new net TG2B_TX: U2.5 (IO5)
- new net TG2_RX: U2.6 (IO6)
- new net USBDM: J5.A7 (D-), J5.B7 (D-), U2.13 (USB_D-)
- new net USBDP: J5.A6 (D+), J5.B6 (D+), U2.14 (USB_D+)
- no-connect marks 0 -> 7
