File: YC265A0-Debug/YC265A0-Debug.kicad_sch (KiCad schematic)
At the start: 0 parts

Commit message: progress
Parts:
- added B1: SPR_DT_SHLD, Connector_JST:JST_SHD_BM40B-SRDS-A-G-TF_2x20-1MP_P1.0mm_Vertical, symbol SPR-DT:SPR_DT_SHLD
- added J1: SPR_DT_BC, parts:CON_528850474_MOL, symbol SPR-DT:SPR_DT_BC
Connections:
- new net +3.3V: J1.1 (+3.3VDSW), J1.15 (+5D), J1.16 (+5D), J1.2 (+3.3VDSW), J1.3 (+3.3VDSW), J1.4 (+3.3VDSW), J1.5 (+3.3VDSW), J1.6 (+3.3VDSW)
- new net BCLK: J1.28 (BICK)
- new net DIN: J1.24 (I2S-PRE)
- new net DOUT: J1.21 (I2S-MIC)
- new net GND: B1.10 (DGND), B1.16 (DGND), B1.21 (DGND), B1.26 (DGND), B1.30 (DGND), B1.34 (DGND), B1.37 (DGND), B1.38 (DGND), B1.4 (DGND), B1.9 (DGND), J1.11 (GND), J1.12 (GND), J1.13 (GND), J1.14 (GND), J1.17 (GND), J1.18 (GND), J1.23 (GND), J1.26 (GND), J1.30 (GND), J1.36 (GND), J1.8 (GND)
- new net MCLK: J1.29 (MCLK)
- new net MIDI-RX0: B1.22 (ACIA-RXD0)
- new net MIDI-RX1: B1.24 (ACIA-RXD1)
- new net MIDI-RX2: B1.27 (ACIA-RXD2)
- new net MIDI-RX3: B1.31 (ACIA-RXD3)
- new net MIDI-TX0: B1.23 (ACIA-TXD0)
- new net MIDI-TX1: B1.25 (ACIA-TXD1)
- new net MIDI-TX2: B1.28 (ACIA-TXD2)
- new net MIDI-TX3: B1.29 (ACIA-TXD3)
- new net MIDI-TX4: B1.32 (ACIA-TXD4)
- new net MIDI-TX5: B1.33 (ACIA-TXD5)
- new net WCLK: J1.27 (LRCK)
- no-connect marks 0 -> 24
Other:
- added sheet AUDIO_IO (AUDIO_IO.kicad_sch)
- added sheet MCU (MCU.kicad_sch)
- title: (none) -> YC265A0 Debugger Board

Commit message: sample 1
Parts:
- added J6: PWR5V, Connector_JST:JST_PH_S4B-PH-SM4-TB_1x04-1MP_P2.00mm_Horizontal, symbol Connector:Conn_01x04_Pin
- added JP3: TDMO0, Connector_PinHeader_2.54mm:PinHeader_1x02_P2.54mm_Vertical, symbol Jumper:Jumper_2_Open
- added JP4: TDMO1, Connector_PinHeader_2.54mm:PinHeader_1x02_P2.54mm_Vertical, symbol Jumper:Jumper_2_Open
- added JP5: TDMI0, Connector_PinHeader_2.54mm:PinHeader_1x02_P2.54mm_Vertical, symbol Jumper:Jumper_2_Open
- added JP6: TDMI1, Connector_PinHeader_2.54mm:PinHeader_1x02_P2.54mm_Vertical, symbol Jumper:Jumper_2_Open
- B1: footprint Connector_JST:JST_SHD_BM40B-SRDS-A-G-TF_2x20-1MP_P1.0mm_Vertical -> parts:JST_SHD_SM40B-SRDS-G-TF_2x20_P1.0_Right_Angle
- J1: footprint parts:CON_528850474_MOL -> parts:529010474
Connections:
- net GND: now also J6.3 (Pin_3), J6.4 (Pin_4)
- net I2S_ADPCM: now reaches B1.11 (SDO-ADPCM)
- net I2S_MP3_0: now reaches B1.13 (SDO-MP3-0)
- net I2S_MP3_1: now reaches B1.14 (SDO-MP3-1)
- net TDMO0: now reaches B1.17 (TDMO-DVNC0)
- net TDMO0: now also JP3.1 (A)
- net TDMO1: now reaches B1.18 (TDMO-DVNC1)
- net TDMO1: now also JP4.1 (A)
- net TDMI0: now reaches B1.19 (TDMI-DVNC0)
- net TDMI0: now also JP5.1 (A)
- net TDMI1: now reaches B1.20 (TDMI-DVNC1)
- net TDMI1: now also JP6.1 (A)
- net I2S_WCLK_MCU: now reaches B1.5 (WCLK-DT)
- net I2S_BCLK_MCU: now reaches B1.6 (BCLK-DT)
- net I2S_MCLK_MCU: now reaches B1.8 (MCLK-DT)
- new net +5V: J6.1 (Pin_1), J6.2 (Pin_2)
- new net I2S_IN: JP3.2 (B), JP4.2 (B), JP5.2 (B), JP6.2 (B)
- no-connect marks 24 -> 26
Other:
- sheet AUDIO_IO ports: added BCLK, DIN, DOUT, MCLK, RESET, SCL, SDA, WCLK; removed CODEC-BCLK, CODEC-DIN, CODEC-DOUT, CODEC-MCLK, CODEC-RESET, CODEC-SCL, CODEC-SDA, CODEC-WCLK
- sheet MCU ports: added CODEC_RESET, I2C_SCL, I2C_SDA, I2S_BCLK, I2S_IN, I2S_MCLK, I2S_OUT1, I2S_OUT2, I2S_OUT3, I2S_WCLK, KDSP_RX, KDSP_TX, SDSP_RX, SDSP_TX, TG1A_TX, TG1B_TX, TG1_RX, TG2A_TX, TG2B_TX, TG2_RX; removed none
